File: 2057-ICE40HX4K-TQ144-breakout.kicad_sch (KiCad schematic)
At the start: 75 parts, among them J1 Conn_02x30_Odd_Even, J2 Conn_02x30_Odd_Even, J3 RaspberryPI-B+header, J4 USB4105-GF-A, J5 RaspberryPI-B+header, J6 Conn_02x08_Odd_Even, J7 Conn_02x01, J8 Micro_SD_Card_Det, U1 ICE40HX4K-TQ144, U2 AZ1117CH-3.3TRG1, U3 AZ1117CH-1.2, U4 AT45DB081E, Y1 XLH536025_000000I

Commit message: Fix DRC error: Unify +3.3V and +3V3 nets
Connections:
- net +3.3V is gone; now on net +3V3: C19.1, C26.1, C27.1, J1.59 (Pin_59), J1.60 (Pin_60), J2.59 (Pin_59), J2.60 (Pin_60), J8.4 (VDD), R10.1, R11.1, R12.1, R13.1, R14.1, R6.1, R7.1, R8.1, R9.1, U2.2 (VO), Y1.4 (VDD)
